Commit message: Added the map_server node to the launch and corrected hokuyo position

File: description/urdf/pioneer3at.urdf (robot description, URDF)
Before this commit: robot pioneer3at, 17 links, 16 joints
Joints:
- joint hokuyo_joint: origin xyz=0.08 0 0.31 rpy=0 0 0 -> xyz=0.28 0 0.31 rpy=0 0 0

Commit message: Just added some comments, nothing important

File: description/urdf/pioneer3at.urdf (robot description, URDF)
Before this commit: robot pioneer3at, 17 links, 16 joints
Joints:
- joint base_top_joint: origin xyz=0.003 0 0.274 rpy=0 0 0 -> xyz=0 0 0.378 rpy=0 0 0
- joint hokuyo_joint: origin xyz=0.28 0 0.31 rpy=0 0 0 -> xyz=0.255 0 0.418 rpy=0 0 0

Commit message: Corrected lidar position

File: description/urdf/pioneer3at.urdf (robot description, URDF)
Before this commit: robot pioneer3at, 17 links, 16 joints
Joints:
- joint hokuyo_joint: origin xyz=0.255 0 0.418 rpy=0 0 0 -> xyz=0.28 0 0.31 rpy=0 0 0

Commit message: Corrected local costmap bug related to laser position (urdf) and voxels

File: description/urdf/pioneer3at.urdf (robot description, URDF)
Before this commit: robot pioneer3at, 17 links, 16 joints
Joints:
- joint hokuyo_joint: origin xyz=0.28 0 0.31 rpy=0 0 0 -> xyz=0.25 0 0.31 rpy=0 0 0
