Commit message: Added sick urdf information to pioneer3at urdf

File: butia_navigation_description/urdf/pioneer3at.urdf (robot description, URDF)
Before this commit: robot pioneer3at, 17 links, 16 joints
Links:
- added link sick_laser, mass 0.001
- added link sick_mount_link, mass 1.1; collision mesh filename=package://butia_navigation_description/meshes/sensors/LMS1x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; visual mesh filename=package://butia_navigation_description/meshes/sensors/LMS1x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
Joints:
- added joint sick_joint: type fixed, parent sick_mount_link, child sick_laser, origin xyz=0.0549 0 0.0367 rpy=0 0 0

Commit message: Changed sick link parameter

File: butia_navigation_description/urdf/pioneer3at.urdf (robot description, URDF)
Before this commit: robot pioneer3at, 19 links, 17 joints
Joints:
- added joint sick_mount_joint: type fixed, parent base_link, child sick_mount_link, origin xyz=0.108 0 0.28 rpy=0 0 0
- joint hokuyo_joint: origin xyz=0.25 0 0.31 rpy=0 0 0 -> xyz=0.08 0 -0.03 rpy=3.1415 0 0

Commit message: Changed hokuyo_link parameters

File: butia_navigation_description/urdf/pioneer3at.urdf (robot description, URDF)
Before this commit: robot pioneer3at, 17 links, 16 joints
Joints:
- joint hokuyo_joint: origin xyz=0.25 0 0.31 rpy=0 0 0 -> xyz=0.08 0 -0.03 rpy=3.1415 0 0

Commit message: Started the tf tree of v3.0 and changed some parameters at costmap params

File: butia_navigation_description/urdf/pioneer3at.urdf (robot description, URDF)
Before this commit: robot pioneer3at, 17 links, 16 joints
Joints:
- joint hokuyo_joint: origin xyz=0.08 0 -0.03 rpy=3.1415 0 0 -> xyz=0.08 0 0.06 rpy=3.1415 0 0

Commit message: Rotated hokuyo_link pi degrees in roll and changed its height in z

File: butia_navigation_description/urdf/pioneer3at.urdf (robot description, URDF)
Before this commit: robot pioneer3at, 17 links, 16 joints
Joints:
- joint hokuyo_joint: origin xyz=0.25 0 0.31 rpy=0 0 0 -> xyz=0.25 0 0.03 rpy=3.1415 0 0

Commit message: Last version in notebook

File: butia_navigation_description/urdf/pioneer3at.urdf (robot description, URDF)
Before this commit: robot pioneer3at, 19 links, 18 joints
Links:
- removed link sick_laser
- added link sick_link, mass 0.001
Joints:
- joint sick_joint: child sick_laser -> sick_link; origin xyz=0.0549 0 0.0367 rpy=0 0 0 -> xyz=0.0549 0 0.12 rpy=0 0 0
- joint sick_mount_joint: origin xyz=0.108 0 0.28 rpy=0 0 0 -> xyz=0.2945 0 0.638 rpy=0 0 0

Commit message: Modified robot mass and inflation rate

File: butia_navigation_description/urdf/pioneer3at.urdf (robot description, URDF)
Before this commit: robot pioneer3at, 19 links, 18 joints
Links:
- link base_link: mass 0.1 -> 60

Commit message: Created a test environment map for simulation

File: butia_navigation_description/urdf/pioneer3at.urdf (robot description, URDF)
Before this commit: robot pioneer3at, 19 links, 18 joints
Links:
- link base_link: mass 60 -> 0.1
- link sick_mount_link: mass 1.1 -> None
Joints:
- joint hokuyo_joint: origin xyz=0.25 0 0.03 rpy=3.1415 0 0 -> xyz=0.25 0 0.06 rpy=3.1415 0 0
- joint sick_mount_joint: origin xyz=0.2945 0 0.638 rpy=0 0 0 -> xyz=0.2945 0 0.38 rpy=0 0 0
