Commit message: Cleaned packages and updated files to reflect new package names

File: butia_navigation_description/urdf/hokuyo.urdf.xacro (robot description, xacro)
@@ -12,5 +12,5 @@
         <origin xyz="0 0 0" rpy="0 0 0"/>
         <geometry>
-          <mesh filename="package://amr_robots_description/meshes/sensors/hokuyo.dae"/>
+          <mesh filename="package://butia_navigation_description/meshes/sensors/hokuyo.dae"/>
         </geometry>
       </visual>

File: butia_navigation_description/urdf/pioneer3at.urdf (robot description, URDF)
Before this commit: robot pioneer3at, 17 links, 16 joints
Links:
- link back_sonar: geometry visual mesh filename=package://butia_navigation_description/meshes/p3at_meshes/b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
- link base_link: geometry collision mesh filename=package://butia_navigation_description/meshes/p3at_meshes/c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; visual mesh filename=package://butia_navigation_description/meshes/p3at_meshes/c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
- link front_sonar: geometry visual mesh filename=package://butia_navigation_description/meshes/p3at_meshes/f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
- link hokuyo_link: geometry collision box size=0.1 0.1 0.1; visual mesh filename=package://butia_navigation_description/meshes/sensors/hokuy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
- link p3at_back_left_axle: geometry collision mesh filename=package://butia_navigation_description/meshes/p3at_meshes/a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; visual mesh filename=package://butia_navigation_description/meshes/p3at_meshes/a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
- link p3at_back_left_hub: geometry collision mesh filename=package://butia_navigation_description/meshes/p3at_meshes/l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; visual mesh filename=package://butia_navigation_description/meshes/p3at_meshes/l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
- link p3at_back_left_wheel: geometry collision cylinder length=0.075 radius=0.111; visual mesh filename=package://butia_navigation_description/meshes/p3at_meshes/w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
- link p3at_back_right_axle: geometry collision mesh filename=package://butia_navigation_description/meshes/p3at_meshes/a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; visual mesh filename=package://butia_navigation_description/meshes/p3at_meshes/a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
- link p3at_back_right_hub: geometry collision mesh filename=package://butia_navigation_description/meshes/p3at_meshes/r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; visual mesh filename=package://butia_navigation_description/meshes/p3at_meshes/r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
- link p3at_back_right_wheel: geometry collision cylinder length=0.075 radius=0.111; visual mesh filename=package://butia_navigation_description/meshes/p3at_meshes/w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
- link p3at_front_left_axle: geometry visual mesh filename=package://butia_navigation_description/meshes/p3at_meshes/a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
- link p3at_front_left_hub: geometry visual mesh filename=package://butia_navigation_description/meshes/p3at_meshes/l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
- link p3at_front_left_wheel: geometry collision cylinder length=0.075 radius=0.111; visual mesh filename=package://butia_navigation_description/meshes/p3at_meshes/w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
- link p3at_front_right_axle: geometry visual mesh filename=package://butia_navigation_description/meshes/p3at_meshes/a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
- link p3at_front_right_hub: geometry visual mesh filename=package://butia_navigation_description/meshes/p3at_meshes/r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
- link p3at_front_right_wheel: geometry collision cylinder length=0.075 radius=0.111; visual mesh filename=package://butia_navigation_description/meshes/p3at_meshes/w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
- link top_plate: geometry visual mesh filename=package://butia_navigation_description/meshes/p3at_meshes/t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

File: butia_navigation_description/urdf/pioneer3at.urdf.xacro (robot description, xacro)
@@ -24,5 +24,5 @@
 			<origin xyz="0 0 0.177" rpy="0 0 0"/>
 			<geometry name="pioneer_geom">
-				<mesh filename="package://amr_robots_description/meshes/p3at_meshes/chassis.stl"/>
+				<mesh filename="package://butia_navigation_description/meshes/p3at_meshes/chassis.stl"/>
 			</geometry>
 			<material name="ChassisRed">
@@ -33,5 +33,5 @@
 			<origin xyz="0 0 0.177" rpy="0 0 0"/>
 				<geometry>
-					<mesh filename="package://amr_robots_description/meshes/p3at_meshes/chassis.stl"/>
+					<mesh filename="package://butia_navigation_description/meshes/p3at_meshes/chassis.stl"/>
 				</geometry>
 		</collision>
@@ -52,5 +52,5 @@
 			<origin xyz="0 0 0" rpy="0 0 0"/>
 			<geometry name="pioneer_geom">
-				<mesh filename="package://amr_robots_description/meshes/p3at_meshes/top.stl"/>
+				<mesh filename="package://butia_navigation_description/meshes/p3at_meshes/top.stl"/>
 			</geometry>
 			<material name="TopBlack">
@@ -78,5 +78,5 @@
 			<origin xyz="0 0 0" rpy="0 0 0"/>
 			<geometry name="pioneer_geom">
-				<mesh filename="package://amr_robots_description/meshes/p3at_meshes/front_sonar.stl"/>
+				<mesh filename="package://butia_navigation_description/meshes/p3at_meshes/front_sonar.stl"/>
 			</geometry>
 			<material name="SonarYellow">
@@ -103,5 +103,5 @@
 			<origin xyz="0 0 0" rpy="0 0 0"/>
 			<geometry name="pioneer_geom">
-				<mesh filename="package://amr_robots_description/meshes/p3at_meshes/back_sonar.stl"/>
+				<mesh filename="package://butia_navigation_description/meshes/p3at_meshes/back_sonar.stl"/>
 			</geometry>
 			<material name="SonarYellow">
@@ -130,5 +130,5 @@
 		<origin xyz="0 0 0" rpy="0 0 0"/>
 		<geometry name="pioneer_geom">
-			<mesh filename="package://amr_robots_description/meshes/p3at_meshes/axle.stl"/>
+			<mesh filename="package://butia_navigation_description/meshes/p3at_meshes/axle.stl"/>
 		</geometry>
 		<material name="AxleGrey">
@@ -155,5 +155,5 @@
 		<origin xyz="0 0 0" rpy="0 0 0"/>
 		<geometry name="pioneer_geom">
-			<mesh filename="package://amr_robots_description/meshes/p3at_meshes/${side}_hubcap.stl"/>
+			<mesh filename="package://butia_navigation_description/meshes/p3at_meshes/${side}_hubcap.stl"/>
 		</geometry>
 		<material name="HubcapYellow">
@@ -180,5 +180,5 @@
 		<origin xyz="0 0 0" rpy="0 0 0"/>
 		<geometry name="pioneer_geom">
-			<mesh filename="package://amr_robots_description/meshes/p3at_meshes/wheel.stl"/>
+			<mesh filename="package://butia_navigation_description/meshes/p3at_meshes/wheel.stl"/>
 		</geometry>
 		<material name="WheelBlack">
@@ -189,5 +189,5 @@
 		<origin xyz="0 0 0" rpy="${-3.1415927/2} 0 0"/>
 		<geometry>
-	    <!--mesh filename="package://amr_robots_description/meshes/p3at_meshes/wheel.stl"/-->
+	    <!--mesh filename="package://butia_navigation_description/meshes/p3at_meshes/wheel.stl"/-->
 	    <cylinder radius="0.111" length="0.075"/>
 		</geometry>
@@ -217,5 +217,5 @@
 		<origin xyz="0 0 0" rpy="0 0 0"/>
 		<geometry name="pioneer_geom">
-			<mesh filename="package://amr_robots_description/meshes/p3at_meshes/axle.stl"/>
+			<mesh filename="package://butia_navigation_description/meshes/p3at_meshes/axle.stl"/>
 		</geometry>
 		<material name="AxleGrey">
@@ -226,5 +226,5 @@
 		<origin xyz="0 0 0" rpy="0 0 0"/>
 		<geometry>
-			<mesh filename="package://amr_robots_description/meshes/p3at_meshes/axle.stl"/>
+			<mesh filename="package://butia_navigation_description/meshes/p3at_meshes/axle.stl"/>
 		</geometry>
 	</collision>
@@ -248,5 +248,5 @@
 		<origin xyz="0 0 0" rpy="0 0 0"/>
 		<geometry name="pioneer_geom">
-			<mesh filename="package://amr_robots_description/meshes/p3at_meshes/${side}_hubcap.stl"/>
+			<mesh filename="package://butia_navigation_description/meshes/p3at_meshes/${side}_hubcap.stl"/>
 		</geometry>
 		<material name="HubcapYellow"/>
@@ -255,5 +255,5 @@
 		<origin xyz="0 0 0" rpy="0 0 0"/>
 		<geometry>
-			<mesh filename="package://amr_robots_description/meshes/p3at_meshes/${side}_hubcap.stl"/>
+			<mesh filename="package://butia_navigation_description/meshes/p3at_meshes/${side}_hubcap.stl"/>
 		</geometry>
 	</collision>
@@ -278,5 +278,5 @@
 		<origin xyz="0 0 0" rpy="0 0 0"/>
 		<geometry name="pioneer_geom">
-			<mesh filename="package://amr_robots_description/meshes/p3at_meshes/wheel.stl"/>
+			<mesh filename="package://butia_navigation_description/meshes/p3at_meshes/wheel.stl"/>
 		</geometry>
 		<material name="WheelBlack"/>
@@ -285,5 +285,5 @@
 		<origin xyz="0 0 0" rpy="${-3.1415927/2} 0 0"/>
 		<geometry>
-	    <!--mesh filename="package://amr_robots_description/meshes/p3at_meshes/wheel.stl"/-->
+	    <!--mesh filename="package://butia_navigation_description/meshes/p3at_meshes/wheel.stl"/-->
 	    <cylinder radius="0.111" length="0.075"/>
 		</geometry>
@@ -397,5 +397,5 @@
   </xacro:macro>
 <!-- Include Hokuyo Laser Sensor and set link -->
-<xacro:include filename="$(find amr_robots_description)/urdf/hokuyo.urdf.xacro"/>
+<xacro:include filename="$(find butia_navigation_description)/urdf/hokuyo.urdf.xacro"/>
 <sensor_hokuyo parent="base_link"/>
 </robot>

File: butia_navigation_description/urdf/pioneer3at_body.xacro (robot description, xacro)
@@ -17,5 +17,5 @@
 			<origin xyz="0 0 0.177" rpy="0 0 0"/>
 			<geometry name="pioneer_geom">
-				<mesh filename="package://amr_robots_description/meshes/p3at_meshes/chassis.stl"/>
+				<mesh filename="package://butia_navigation_description/meshes/p3at_meshes/chassis.stl"/>
 			</geometry>
 			<material name="ChassisRed">
@@ -26,5 +26,5 @@
 			<origin xyz="0 0 0.177" rpy="0 0 0"/>
 				<geometry>
-					<mesh filename="package://amr_robots_description/meshes/p3at_meshes/chassis.stl"/>
+					<mesh filename="package://butia_navigation_description/meshes/p3at_meshes/chassis.stl"/>
 				</geometry>
 		</collision>
@@ -45,5 +45,5 @@
 			<origin xyz="0 0 0" rpy="0 0 0"/>
 			<geometry name="pioneer_geom">
-				<mesh filename="package://amr_robots_description/meshes/p3at_meshes/top.stl"/>
+				<mesh filename="package://butia_navigation_description/meshes/p3at_meshes/top.stl"/>
 			</geometry>
 			<material name="TopBlack">
@@ -71,5 +71,5 @@
 			<origin xyz="0 0 0" rpy="0 0 0"/>
 			<geometry name="pioneer_geom">
-				<mesh filename="package://amr_robots_description/meshes/p3at_meshes/front_sonar.stl"/>
+				<mesh filename="package://butia_navigation_description/meshes/p3at_meshes/front_sonar.stl"/>
 			</geometry>
 			<material name="SonarYellow">
@@ -96,5 +96,5 @@
 			<origin xyz="0 0 0" rpy="0 0 0"/>
 			<geometry name="pioneer_geom">
-				<mesh filename="package://amr_robots_description/meshes/p3at_meshes/back_sonar.stl"/>
+				<mesh filename="package://butia_navigation_description/meshes/p3at_meshes/back_sonar.stl"/>
 			</geometry>
 			<material name="SonarYellow">
@@ -123,5 +123,5 @@
 		<origin xyz="0 0 0" rpy="0 0 0"/>
 		<geometry name="pioneer_geom">
-			<mesh filename="package://amr_robots_description/meshes/p3at_meshes/axle.stl"/>
+			<mesh filename="package://butia_navigation_description/meshes/p3at_meshes/axle.stl"/>
 		</geometry>
 		<material name="AxleGrey">
@@ -148,5 +148,5 @@
 		<origin xyz="0 0 0" rpy="0 0 0"/>
 		<geometry name="pioneer_geom">
-			<mesh filename="package://amr_robots_description/meshes/p3at_meshes/${suffix}_hubcap.stl"/>
+			<mesh filename="package://butia_navigation_description/meshes/p3at_meshes/${suffix}_hubcap.stl"/>
 		</geometry>
 		<material name="HubcapYellow">
@@ -173,5 +173,5 @@
 		<origin xyz="0 0 0" rpy="0 0 0"/>
 		<geometry name="pioneer_geom">
-			<mesh filename="package://amr_robots_description/meshes/p3at_meshes/wheel.stl"/>
+			<mesh filename="package://butia_navigation_description/meshes/p3at_meshes/wheel.stl"/>
 		</geometry>
 		<material name="WheelBlack">
@@ -182,5 +182,5 @@
 		<origin xyz="0 0 0" rpy="${-3.1415927/2} 0 0"/>
 		<geometry>
-	    <!--mesh filename="package://amr_robots_description/meshes/p3at_meshes/wheel.stl"/-->
+	    <!--mesh filename="package://butia_navigation_description/meshes/p3at_meshes/wheel.stl"/-->
 	    <cylinder radius="0.111" length="0.075"/>
 		</geometry>
@@ -210,5 +210,5 @@
 		<origin xyz="0 0 0" rpy="0 0 0"/>
 		<geometry name="pioneer_geom">
-			<mesh filename="package://amr_robots_description/meshes/p3at_meshes/axle.stl"/>
+			<mesh filename="package://butia_navigation_description/meshes/p3at_meshes/axle.stl"/>
 		</geometry>
 		<material name="AxleGrey">
@@ -219,5 +219,5 @@
 		<origin xyz="0 0 0" rpy="0 0 0"/>
 		<geometry>
-			<mesh filename="package://amr_robots_description/meshes/p3at_meshes/axle.stl"/>
+			<mesh filename="package://butia_navigation_description/meshes/p3at_meshes/axle.stl"/>
 		</geometry>
 	</collision>
@@ -241,5 +241,5 @@
 		<origin xyz="0 0 0" rpy="0 0 0"/>
 		<geometry name="pioneer_geom">
-			<mesh filename="package://amr_robots_description/meshes/p3at_meshes/${suffix}_hubcap.stl"/>
+			<mesh filename="package://butia_navigation_description/meshes/p3at_meshes/${suffix}_hubcap.stl"/>
 		</geometry>
 		<material name="HubcapYellow"/>
@@ -248,5 +248,5 @@
 		<origin xyz="0 0 0" rpy="0 0 0"/>
 		<geometry>
-			<mesh filename="package://amr_robots_description/meshes/p3at_meshes/${suffix}_hubcap.stl"/>
+			<mesh filename="package://butia_navigation_description/meshes/p3at_meshes/${suffix}_hubcap.stl"/>
 		</geometry>
 	</collision>
@@ -270,5 +270,5 @@
 		<origin xyz="0 0 0" rpy="0 0 0"/>
 		<geometry name="pioneer_geom">
-			<mesh filename="package://amr_robots_description/meshes/p3at_meshes/wheel.stl"/>
+			<mesh filename="package://butia_navigation_description/meshes/p3at_meshes/wheel.stl"/>
 		</geometry>
 		<material name="WheelBlack"/>
@@ -277,5 +277,5 @@
 		<origin xyz="0 0 0" rpy="${-3.1415927/2} 0 0"/>
 		<geometry>
-	    <!--mesh filename="package://amr_robots_description/meshes/p3at_meshes/wheel.stl"/-->
+	    <!--mesh filename="package://butia_navigation_description/meshes/p3at_meshes/wheel.stl"/-->
 	    <cylinder radius="0.111" length="0.075"/>
 		</geometry>

File: butia_navigation_description/urdf/pioneer3at_hokuyo.urdf.xacro (robot description, xacro)
@@ -24,5 +24,5 @@
 			<origin xyz="0 0 0.177" rpy="0 0 0"/>
 			<geometry name="pioneer_geom">
-				<mesh filename="package://amr_robots_description/meshes/p3at_meshes/chassis.stl"/>
+				<mesh filename="package://butia_navigation_description/meshes/p3at_meshes/chassis.stl"/>
 			</geometry>
 			<material name="ChassisRed">
@@ -33,5 +33,5 @@
 			<origin xyz="0 0 0.177" rpy="0 0 0"/>
 				<geometry>
-					<mesh filename="package://amr_robots_description/meshes/p3at_meshes/chassis.stl"/>
+					<mesh filename="package://butia_navigation_description/meshes/p3at_meshes/chassis.stl"/>
 				</geometry>
 		</collision>
@@ -52,5 +52,5 @@
 			<origin xyz="0 0 0" rpy="0 0 0"/>
 			<geometry name="pioneer_geom">
-				<mesh filename="package://amr_robots_description/meshes/p3at_meshes/top.stl"/>
+				<mesh filename="package://butia_navigation_description/meshes/p3at_meshes/top.stl"/>
 			</geometry>
 			<material name="TopBlack">
@@ -78,5 +78,5 @@
 			<origin xyz="0 0 0" rpy="0 0 0"/>
 			<geometry name="pioneer_geom">
-				<mesh filename="package://amr_robots_description/meshes/p3at_meshes/front_sonar.stl"/>
+				<mesh filename="package://butia_navigation_description/meshes/p3at_meshes/front_sonar.stl"/>
 			</geometry>
 			<material name="SonarYellow">
@@ -103,5 +103,5 @@
 			<origin xyz="0 0 0" rpy="0 0 0"/>
 			<geometry name="pioneer_geom">
-				<mesh filename="package://amr_robots_description/meshes/p3at_meshes/back_sonar.stl"/>
+				<mesh filename="package://butia_navigation_description/meshes/p3at_meshes/back_sonar.stl"/>
 			</geometry>
 			<material name="SonarYellow">
@@ -130,5 +130,5 @@
 		<origin xyz="0 0 0" rpy="0 0 0"/>
 		<geometry name="pioneer_geom">
-			<mesh filename="package://amr_robots_description/meshes/p3at_meshes/axle.stl"/>
+			<mesh filename="package://butia_navigation_description/meshes/p3at_meshes/axle.stl"/>
 		</geometry>
 		<material name="AxleGrey">
@@ -155,5 +155,5 @@
 		<origin xyz="0 0 0" rpy="0 0 0"/>
 		<geometry name="pioneer_geom">
-			<mesh filename="package://amr_robots_description/meshes/p3at_meshes/${side}_hubcap.stl"/>
+			<mesh filename="package://butia_navigation_description/meshes/p3at_meshes/${side}_hubcap.stl"/>
 		</geometry>
 		<material name="HubcapYellow">
@@ -180,5 +180,5 @@
 		<origin xyz="0 0 0" rpy="0 0 0"/>
 		<geometry name="pioneer_geom">
-			<mesh filename="package://amr_robots_description/meshes/p3at_meshes/wheel.stl"/>
+			<mesh filename="package://butia_navigation_description/meshes/p3at_meshes/wheel.stl"/>
 		</geometry>
 		<material name="WheelBlack">
@@ -189,5 +189,5 @@
 		<origin xyz="0 0 0" rpy="${-3.1415927/2} 0 0"/>
 		<geometry>
-	    <!--mesh filename="package://amr_robots_description/meshes/p3at_meshes/wheel.stl"/-->
+	    <!--mesh filename="package://butia_navigation_description/meshes/p3at_meshes/wheel.stl"/-->
 	    <cylinder radius="0.111" length="0.075"/>
 		</geometry>
@@ -217,5 +217,5 @@
 		<origin xyz="0 0 0" rpy="0 0 0"/>
 		<geometry name="pioneer_geom">
-			<mesh filename="package://amr_robots_description/meshes/p3at_meshes/axle.stl"/>
+			<mesh filename="package://butia_navigation_description/meshes/p3at_meshes/axle.stl"/>
 		</geometry>
 		<material name="AxleGrey">
@@ -226,5 +226,5 @@
 		<origin xyz="0 0 0" rpy="0 0 0"/>
 		<geometry>
-			<mesh filename="package://amr_robots_description/meshes/p3at_meshes/axle.stl"/>
+			<mesh filename="package://butia_navigation_description/meshes/p3at_meshes/axle.stl"/>
 		</geometry>
 	</collision>
@@ -248,5 +248,5 @@
 		<origin xyz="0 0 0" rpy="0 0 0"/>
 		<geometry name="pioneer_geom">
-			<mesh filename="package://amr_robots_description/meshes/p3at_meshes/${side}_hubcap.stl"/>
+			<mesh filename="package://butia_navigation_description/meshes/p3at_meshes/${side}_hubcap.stl"/>
 		</geometry>
 		<material name="HubcapYellow"/>
@@ -255,5 +255,5 @@
 		<origin xyz="0 0 0" rpy="0 0 0"/>
 		<geometry>
-			<mesh filename="package://amr_robots_description/meshes/p3at_meshes/${side}_hubcap.stl"/>
+			<mesh filename="package://butia_navigation_description/meshes/p3at_meshes/${side}_hubcap.stl"/>
 		</geometry>
 	</collision>
@@ -278,5 +278,5 @@
 		<origin xyz="0 0 0" rpy="0 0 0"/>
 		<geometry name="pioneer_geom">
-			<mesh filename="package://amr_robots_description/meshes/p3at_meshes/wheel.stl"/>
+			<mesh filename="package://butia_navigation_description/meshes/p3at_meshes/wheel.stl"/>
 		</geometry>
 		<material name="WheelBlack"/>
@@ -285,5 +285,5 @@
 		<origin xyz="0 0 0" rpy="${-3.1415927/2} 0 0"/>
 		<geometry>
-	    <!--mesh filename="package://amr_robots_description/meshes/p3at_meshes/wheel.stl"/-->
+	    <!--mesh filename="package://butia_navigation_description/meshes/p3at_meshes/wheel.stl"/-->
 	    <cylinder radius="0.111" length="0.075"/>
 		</geometry>
@@ -395,5 +395,5 @@
   </xacro:macro>
 <!--  Hokuyo Laser Sensor-->
-<xacro:include filename="$(find amr_robots_description)/urdf/hokuyo.urdf.xacro"/>
+<xacro:include filename="$(find butia_navigation_description)/urdf/hokuyo.urdf.xacro"/>
 <sensor_hokuyo parent="base_link"/>
 </robot>

Commit message: fixing some things for real robot and new maps

File: butia_navigation_description/urdf/hokuyo.urdf.xacro (robot description, xacro)
@@ -23,5 +23,5 @@
     <joint name="hokuyo_joint" type="fixed">
       <!--<axis xyz="0 0 1" />-->
-      <origin xyz="0.08 0 0.31" rpy="0 0 0"/>
+      <origin xyz="0.08 0 0.31" rpy="3.14 0 0"/>
       <parent link="${parent}"/>
       <child link="hokuyo_link"/>
