Commit message: Corrected distances

File: butia_navigation_description/urdf/v2.0/pioneer3at.urdf (robot description, URDF)
Before this commit: robot pioneer3at, 19 links, 18 joints
Links:
- link base_link: mass 0.1 -> 60
- link sick_mount_link: mass None -> 1.1
Joints:
- joint base_top_joint: origin xyz=0.003 0 0.274 rpy=0 0 0 -> xyz=0 0 0.378 rpy=0 0 0
- joint hokuyo_joint: origin xyz=0.25 0 0.06 rpy=3.1415 0 0 -> xyz=0.25 0 0.03 rpy=3.1415 0 0
- joint sick_mount_joint: origin xyz=0.2945 0 0.38 rpy=0 0 0 -> xyz=0.2945 0 0.638 rpy=0 0 0
